File: hardware/rf_board.sch (EAGLE design)
At the start: 31 parts, among them IC1 LM358MX, X3 KUSBVX

Commit message: RF board update
Connections:
- removed net SCL: U$1.2.CLK
- removed net SDA: U$1.1.DATA
- net SCL1: now also U$1.2.CLK
- net SDA1: now also U$1.1.DATA
Changed lines of the file:
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@@
 <label x="551.18" y="302.26" size="1.4224" layer="95" rot="R180" xref="yes"/>
+</segment>
+<segment>
+<pinref part="U$1" gate="G$1" pin="2.CLK"/>
+<wire x1="436.88" y1="396.24" x2="426.72" y2="396.24" width="0.1524" layer="91"/>
+<label x="426.72" y="396.24" size="1.4224" layer="95" rot="R180" xref="yes"/>
 </segment>
 </net>
@@
 <label x="551.18" y="304.8" size="1.4224" layer="95" rot="R180" xref="yes"/>
 </segment>
+<segment>
+<pinref part="U$1" gate="G$1" pin="1.DATA"/>
+<wire x1="436.88" y1="401.32" x2="426.72" y2="401.32" width="0.1524" layer="91"/>
+<label x="426.72" y="401.32" size="1.4224" layer="95" rot="R180" xref="yes"/>
+</segment>
 </net>
 <net name="RF2_ROT_SW" class="0">
@@
 </segment>
 </net>
-<net name="SDA" class="0">
-<segment>
-<pinref part="U$1" gate="G$1" pin="1.DATA"/>
-<wire x1="436.88" y1="401.32" x2="426.72" y2="401.32" width="0.1524" layer="91"/>
-<label x="426.72" y="401.32" size="1.4224" layer="95" rot="R180" xref="yes"/>
-</segment>
-</net>
-<net name="SCL" class="0">
-<segment>
-<pinref part="U$1" gate="G$1" pin="2.CLK"/>
-<wire x1="436.88" y1="396.24" x2="426.72" y2="396.24" width="0.1524" layer="91"/>
-<label x="426.72" y="396.24" size="1.4224" layer="95" rot="R180" xref="yes"/>
-</segment>
-</net>

Commit message: RF board updated
Parts:
- added C15, C16, C17, C18, C19, C20, C21, C22, C23, C24, C25, C26, C27, C28, C29, C30, C31, C32, C33, C34, C35: (no value), rcl:C-EUC0805
- added C36, C37: 100n, rcl:C-EUC0603
- added L1, L10, L11, L12, L13, L14, L2, L3, L4, L5, L6, L7, L8, L9: (no value), rcl:R-EU_R0805
- added R10: (no value), rcl:R-EU_0204/7
- added R11: (no value), rcl:R-EU_0204/5
- added U$4, U$5: SN74CBT3251, mw:SN74CBT3251
- added X1, X2: SMA-142-0701-801/806, con-coax:SMA-142-0701-801/806
Connections:
- removed net N$12: U$2.SEL1, U$2.SEL2
- removed net RD7: SV1.16
- removed net RG0: SV1.18
- removed net RG1: SV1.15
- new net LPF_16_30_A: C17.1, L2.1, U$5.B4
- new net LPF_16_30_B: C16.1, L1.2, U$4.B4
- new net LPF_1_2_A: C29.1, L10.1, U$5.B5
- new net LPF_1_2_B: C28.1, L9.2, U$4.B5
- new net LPF_250K_A: C35.1, L14.1, U$5.B7
- new net LPF_250K_B: C34.1, L13.2, U$4.B7
- new net LPF_2_4_A: C26.1, L8.1, U$5.B1
- new net LPF_2_4_B: C25.1, L7.2, U$4.B1
- new net LPF_4_8_A: C23.1, L6.1, U$5.B2
- new net LPF_4_8_B: C22.1, L5.2, U$4.B2
- new net LPF_500K_1_A: C32.1, L12.1, U$5.B6
- new net LPF_500K_1_B: C31.1, L11.2, U$4.B6
- new net LPF_8_16_A: C20.1, L4.1, U$5.B3
- new net LPF_8_16_B: C19.1, L3.2, U$4.B3
- new net N$19: C15.1, L1.1, L2.2
- new net N$20: U$5.A, X2.1
- new net N$21: U$1.10.ANT, X1.1
- new net N$22: C18.1, L3.1, L4.2
- new net N$25: C21.1, L5.1, L6.2
- new net N$28: C24.1, L7.1, L8.2
- new net N$31: C27.1, L10.2, L9.1
- new net N$34: C30.1, L11.1, L12.2
- new net N$38: C33.1, L13.1, L14.2
- new net N$41: C9.1, U$4.A
- new net NO_LPF: U$4.B8, U$5.B8
- new net RD7_BAND_A0: SV1.16, U$4.S0, U$5.S0
- new net RG0_BAND_A2: SV1.18, U$4.S2, U$5.S2
- new net RG1_BAND_A1: SV1.15, U$4.S1, U$5.S1
- net 3V: now also R10.2, R11.2
- net RA6: now also U$2.SEL1, U$2.SEL2
- net SCL1: now also R10.1
- net SDA1: now also R11.1
- net VBUS: now also C36.1, C37.1, U$4.VCC, U$5.VCC
- net VS_AGND: now also C15.2, C16.2, C17.2, C18.2, C19.2, C20.2, C21.2, C22.2, C23.2, C24.2, C25.2, C26.2, C27.2, C28.2, C29.2, C30.2, C31.2, C32.2, C33.2, C34.2, C35.2, C36.2, C37.2, U$4.!OE, U$4.GND, U$5.!OE, U$5.GND, X1.2, X2.2
